File: us_sonar_v2_pcb.kicad_pcb (KiCad board)
At the start: 2 copper layers, 17 parts, among them IC1 TUSS4470TRTJT, IC2 Adafruit_BMP085, IC3 MIKROE-HUM&TEMP_21click, IC4 DFRobot_SEN0161, IC5 DS18B20+T&R, IC6 Waveshare_NEO6M, IC7 US_Transceiver

Commit message: version_1_pcb
Parts:
- added C10: 100n, Capacitor_SMD:C_0805_2012Metric, F.Cu at (68.5, 113.0)
- added C11: 100u, Capacitor_THT:CP_Radial_D10.0mm_P5.00mm, F.Cu at (64.0, 118.1)
- added C12: 100n, Capacitor_SMD:C_0805_2012Metric, F.Cu at (100.0, 206.5)
- added C13: 100n, Capacitor_SMD:C_0805_2012Metric, F.Cu at (113.0, 177.0)
- added C14: 100n, Capacitor_SMD:C_0805_2012Metric_Pad1.18x1.45mm_HandSolder, F.Cu at (124.0, 208.5)
- added C15: 100n, Capacitor_SMD:C_0805_2012Metric, F.Cu at (101.0, 156.0)
- added C16: 10u, Capacitor_THT:CP_Radial_D5.0mm_P2.00mm, F.Cu at (107.5, 156.5)
- added C17: C, Capacitor_SMD:C_0805_2012Metric_Pad1.18x1.45mm_HandSolder, F.Cu at (93.0, 179.0)
- added C18: C, Capacitor_SMD:C_0805_2012Metric_Pad1.18x1.45mm_HandSolder, F.Cu at (94.0, 202.5)
- added C7: 10u, Capacitor_SMD:C_0805_2012Metric_Pad1.18x1.45mm_HandSolder, F.Cu at (156.5, 153.0)
- added C8: 22u, Capacitor_SMD:C_0805_2012Metric, F.Cu at (156.5, 158.0)
- added C9: 10u, Capacitor_SMD:C_0805_2012Metric, F.Cu at (113.0, 173.0)
- added IC8: MCP1700-3302E_TO, SamacSys_Parts:MCP17003302ETO, F.Cu at (106.0, 175.0)
- added J2: Conn_01x04_Pin, Connector_PinHeader_2.54mm:PinHeader_1x04_P2.54mm_Vertical, F.Cu at (124.0, 173.3)
- added J3: Conn_01x04_Pin, Connector_PinHeader_2.54mm:PinHeader_1x04_P2.54mm_Vertical, F.Cu at (117.0, 198.0)
- added R4: 4k7, Resistor_SMD:R_0805_2012Metric_Pad1.20x1.40mm_HandSolder, F.Cu at (216.9, 196.1)
- added SW1: SW_MEC_5G, Button_Switch_SMD:SW_MEC_5GSH9, F.Cu at (60.0, 133.5)
- added U1: 18650 2S, SamacSys_Parts:1048, F.Cu at (203.1, 112.0)
- added U2: Charger 18650, SamacSys_Parts:Charger 18650, F.Cu at (124.0, 110.5)
- added U3: BMS + BALANCER, SamacSys_Parts:BMS 2S module, B.Cu at (155.1, 137.4)
- added U4: MT3608, SamacSys_Parts:MT3608_module, F.Cu at (73.0, 113.8)
- added U5: VX07805, SamacSys_Parts:VX07805, F.Cu at (160.5, 155.5)
- A1: value RaspberryPi_Pico_W -> RaspberryPi_Pico; footprint Module:RaspberryPi_Pico_W_SMD -> Module:RaspberryPi_Pico_Common_THT
- C1, C2, C3, C4, C5: footprint Capacitor_SMD:C_0603_1608Metric_Pad1.08x0.95mm_HandSolder -> Capacitor_SMD:C_0805_2012Metric_Pad1.18x1.45mm_HandSolder
- moved A1 215.4 mm to (147.9, 212.8), turned to 180 degrees
- moved IC7 193.4 mm to (56.0, 189.8)
- moved C2 183.9 mm to (100.0, 202.5), turned to -90 degrees
- moved C3 182.0 mm to (97.0, 202.5), turned to -90 degrees
- moved C6 174.2 mm to (98.8, 195.5), turned to 180 degrees
- moved IC4 172.8 mm to (95.2, 158.0), turned to -90 degrees
- moved C1 169.4 mm to (99.0, 185.0), turned to 180 degrees
- moved IC1 169.3 mm to (107.5, 191.5), turned to 90 degrees
- moved R1 169.2 mm to (94.0, 185.0), turned to 180 degrees
- moved IC2 162.0 mm to (189.0, 195.5), turned to 90 degrees
- moved C4 155.9 mm to (100.0, 179.0), turned to 90 degrees
- moved C5 154.2 mm to (96.5, 179.0), turned to 90 degrees
- moved IC5 148.8 mm to (211.9, 195.1), turned to -90 degrees
- moved IC3 147.6 mm to (170.5, 195.5), turned to -90 degrees
- moved R3 142.5 mm to (101.0, 165.0), turned to 90 degrees
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Connections:
- A1 pad 11: /UART1_TX -> unconnected-(A1-GPIO8-Pad11)
- A1 pad 12: /UART1_RX -> unconnected-(A1-GPIO9-Pad12)
- A1 pad 14: unconnected-(A1-GPIO10-Pad14) -> /1WIRE
- A1 pad 16: unconnected-(A1-GPIO12-Pad16) -> /UART0_TX
- A1 pad 17: unconnected-(A1-GPIO13-Pad17) -> /UART0_RX
- A1 pad 20: /1WIRE -> unconnected-(A1-GPIO15-Pad20)
- A1 pad 21: unconnected-(A1-GPIO16-Pad21) -> /SPI0_MISO
- A1 pad 22: unconnected-(A1-GPIO17-Pad22) -> /SPI0_CSn
- A1 pad 24: /BURST -> /SPI0_SCK
- A1 pad 25: unconnected-(A1-GPIO19-Pad25) -> /SPI0_MOSI
- A1 pad 27: unconnected-(A1-GPIO21-Pad27) -> /BURST
- A1 pad 36: /3V3 MCU -> +3V3 MCU
- A1 pad 39: /VSYS -> +5V
- A1 pad 4: /SPI0_SCK -> unconnected-(A1-GPIO2-Pad4)
- A1 pad 40: /VBUS -> unconnected-(A1-VBUS-Pad40)
- A1 pad 5: /SPI0_MOSI -> unconnected-(A1-GPIO3-Pad5)
- A1 pad 6: /SPI0_MISO -> unconnected-(A1-GPIO4-Pad6)
- A1 pad 7: /SPI0_CSn -> unconnected-(A1-GPIO5-Pad7)
- IC1 pad 3: /SPI0_CSn -> /SPI0_CSn_TUSS4470
- IC1 pad 4: /SPI0_SCK -> /SPI0_SCK_TUSS4470
- IC1 pad 5: /SPI0_MOSI -> /SPI0_MOSI_TUSS4470
- IC1 pad 6: /SPI0_MISO -> /SPI0_MISO_TUSS4470
- IC2 pad 1: +3V3 -> +3V3 MCU
- IC3 pad 7: +3V3 -> +3V3 MCU
- IC5 pad 3: +3V3 -> +3V3 MCU
- IC6 pad 2: /UART1_TX -> /UART0_TX
- IC6 pad 3: /UART1_RX -> /UART0_RX
Routing:
- net +5V: track 0.00 -> 214.3 mm, vias 0 -> 1
- net +3V3 MCU: track 0.00 -> 160.4 mm
- net /ADC2_PH_SENSOR: track 0.00 -> 151.6 mm, vias 0 -> 1
- net VBAT: track 0.00 -> 148.3 mm
- net VPWR: track 0.00 -> 135.8 mm, vias 0 -> 1
- net /RST_SW: track 0.00 -> 110.0 mm
- net /1WIRE: track 0.00 -> 75.4 mm
- net Net-(IC1-OUTA): track 0.00 -> 52.5 mm
- net /I2C0_SDA: track 0.00 -> 48.3 mm
- net /I2C0_SCL: track 0.00 -> 48.3 mm
- net /UART0_TX: track 0.00 -> 48.0 mm, vias 0 -> 1
- net Net-(IC1-OUTB): track 0.00 -> 47.9 mm
- net /UART0_RX: track 0.00 -> 45.9 mm
- net Net-(U1-+_2): track 0.00 -> 23.5 mm
- net Net-(U1--_1): track 0.00 -> 23.4 mm
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- added copper zone on B.Cu, net GND
- added copper zone on F.Cu, net GND
Other:
- board outline added: 180 x 117 mm
