File: us_sonar_v2_pcb.kicad_sch (KiCad schematic)
At the start: 17 parts, among them IC1 TUSS4470TRTJT, IC2 Adafruit_BMP085, IC3 MIKROE-HUM&TEMP_21click, IC4 DFRobot_SEN0161, IC5 DS18B20+T&R, IC6 Waveshare_NEO6M, IC7 US_Transceiver

Commit message: version_1_pcb
Parts:
- added C10, C12, C13, C15: 100n, Capacitor_SMD:C_0805_2012Metric, symbol Device:C
- added C11: 100u, Capacitor_THT:CP_Radial_D10.0mm_P5.00mm, symbol Device:C_Polarized
- added C14: 100n, Capacitor_SMD:C_0805_2012Metric_Pad1.18x1.45mm_HandSolder, symbol Device:C
- added C16: 10u, Capacitor_THT:CP_Radial_D5.0mm_P2.00mm, symbol Device:C_Polarized
- added C17, C18: C, Capacitor_SMD:C_0805_2012Metric_Pad1.18x1.45mm_HandSolder, symbol Device:C
- added C7: 10u, Capacitor_SMD:C_0805_2012Metric_Pad1.18x1.45mm_HandSolder, symbol Device:C
- added C8: 22u, Capacitor_SMD:C_0805_2012Metric, symbol Device:C
- added C9: 10u, Capacitor_SMD:C_0805_2012Metric, symbol Device:C
- added IC8: MCP1700-3302E_TO, MCP17003302ETO, symbol SamacSys:MCP1700-3302E_TO
- added J2, J3: Conn_01x04_Pin, Connector_PinHeader_2.54mm:PinHeader_1x04_P2.54mm_Vertical, symbol Connector:Conn_01x04_Pin
- added R4: 4k7, Resistor_SMD:R_0805_2012Metric_Pad1.20x1.40mm_HandSolder, symbol Device:R
- added SW1: SW_MEC_5G, Button_Switch_SMD:SW_MEC_5GSH9, symbol Switch:SW_MEC_5G
- added U1: 18650 2S, SamacSys_Parts:1048, symbol SamacSys:1048
- added U2: Charger 18650, SamacSys_Parts:Charger 18650, symbol SamacSys:Charger_USB-C_18650_2S_2A
- added U3: BMS + BALANCER, SamacSys_Parts:BMS 2S module, symbol SamacSys:BMS_2S_+_balanser_module
- added U4: MT3608, SamacSys_Parts:MT3608_module, symbol SamacSys:MT3608_module
- added U5: VX07805, SamacSys_Parts:VX07805, symbol SamacSys:VX07805
- A1: footprint Module:RaspberryPi_Pico_SMD_HandSolder -> Module:RaspberryPi_Pico_Common_THT
- C1, C2, C3, C4, C5: footprint Capacitor_SMD:C_0603_1608Metric_Pad1.08x0.95mm_HandSolder -> Capacitor_SMD:C_0805_2012Metric_Pad1.18x1.45mm_HandSolder
- C6: symbol Device:C -> Device:C_Polarized
Connections:
- net VSYS is gone; now on net +5V: A1.39 (VSYS)
- net +3V3: now also C13.1, C9.1, IC8.3 (VOUT); no longer IC2.1 (VIN), IC3.7 (3V3), IC5.3 (VDD)
- net +5V: now also C14.1, C15.1, C16.1, C8.1, IC8.2 (VIN), U5.3 (+5V)
- net 1WIRE: now also A1.14 (GPIO10), R4.1; no longer A1.20 (GPIO15)
- net BURST: now also A1.27 (GPIO21); no longer A1.24 (GPIO18)
- net GND: now also C10.2, C11.2, C12.2, C13.2, C14.2, C15.2, C16.2, C17.2, C18.2, C7.2, C8.2, C9.2, IC8.1 (GND), SW1.1 (A), SW1.2 (A), U2.2 (GND), U2.4 (GND), U3.2 (-), U4.2 (VIN-), U4.4 (VOUT-), U5.2 (GND)
- net RST_SW: now also SW1.3 (B), SW1.4 (B)
- net SPI0_CSn: now also A1.22 (GPIO17), J2.3 (Pin_3); no longer A1.7 (GPIO5), IC1.3 (NCS)
- net SPI0_MISO: now also A1.21 (GPIO16), J2.4 (Pin_4); no longer A1.6 (GPIO4), IC1.6 (SDO)
- net SPI0_MOSI: now also A1.25 (GPIO19), J2.1 (Pin_1); no longer A1.5 (GPIO3), IC1.5 (SDI)
- net SPI0_SCK: now also A1.24 (GPIO18), J2.2 (Pin_2); no longer A1.4 (GPIO2), IC1.4 (SCLK)
- net VPWR: now also C10.1, C11.1, C12.1, U4.3 (VOUT+)
- net at C2.1, C3.1, IC1.18 (FLT): now also C18.1
- net at C4.1, C5.1, IC1.11 (INN): now also C17.1
- net UART0_TX: now reaches A1.16 (GPIO12)
- net UART0_TX: now also IC6.2 (RX)
- net UART0_RX: now reaches A1.17 (GPIO13)
- net UART0_RX: now also IC6.3 (TX)
- net 3V3 MCU renamed +3V3 MCU
- net +3V3 MCU: now also IC2.1 (VIN), IC3.7 (3V3), IC5.3 (VDD), R4.2
- net SWCLK: no longer names the net of A1.D1 (SWCLK)
- net SWDIO: no longer names the net of A1.D3 (SWDIO)
- net UART1_RX: no longer names the net of A1.12 (GPIO9)
- net UART1_RX: no longer IC6.3 (TX)
- net UART1_TX: no longer names the net of A1.11 (GPIO8)
- net UART1_TX: no longer IC6.2 (RX)
- net VBUS: no longer names the net of A1.40 (VBUS)
- new net: U1.4 (+_2), U3.3 (8.4V)
- new net: U1.2 (+_1), U1.3 (-_2), U3.4 (4.2V)
- new net: U1.1 (-_1), U3.5 (0V)
- new net SPI0_CSn_TUSS4470: IC1.3 (NCS), J3.1 (Pin_1)
- new net SPI0_MISO_TUSS4470: IC1.6 (SDO), J3.4 (Pin_4)
- new net SPI0_MOSI_TUSS4470: IC1.5 (SDI), J3.3 (Pin_3)
- new net SPI0_SCK_TUSS4470: IC1.4 (SCLK), J3.2 (Pin_2)
- new net VBAT: C7.1, U2.3 (BAT), U3.1 (+), U4.1 (VIN+), U5.1 (Vin)
- new net VCHARGE: U2.1 (Vin)
- no-connect marks 37 -> 39
Other:
- note added: "+3V3 LDO"
- note added: "+5V Regulator"
- note added: "Charger, BMS & Cells"
- note added: "POWER"
- note added: "VPWR Regulator"
- note added: "change firmware to acomodate new pinout"
- moved on the sheet: C4, C5, IC4, IC5, IC6, R2, R3
